File: Hardware/PCB/BatteryBoard/BatteryBoard-backups/BatteryBoard-2023-12-28_211333/BatteryBoard.kicad_pcb (KiCad board)
At the start: 2 copper layers, 60 x 60 mm, 78 parts, among them J1 USB_C_Receptacle_USB2.0, J2 Thermistor, J3 Conn_01x07, J4 Conn_01x07, J5 Conn_01x07, J6 Conn_01x07, J7 Power, Q1 FDS4935A, Q2 FDS4935A, SW1 SW_SPDT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

Commit message: 配線中
Parts:
- C22, C23: value 10u(3216) -> 10u(3225); footprint Capacitor_SMD:C_1206_3216Metric -> Capacitor_SMD:C_1210_3225Metric
- C24, C25: value 22u(3216) -> 22u(3225); footprint Capacitor_SMD:C_1206_3216Metric -> Capacitor_SMD:C_1210_3225Metric
- moved R29 3.14 mm to (130.7, 121.3)
- moved R27 3.06 mm to (130.7, 111.7)
- moved R26 2.96 mm to (129.2, 111.7), turned to 90 degrees
- moved R28 2.54 mm to (129.2, 121.3), turned to 90 degrees
- moved C23 2.09 mm to (126.1, 123.9), turned to 180 degrees
- moved C20 1.55 mm to (132.2, 111.7), turned to 90 degrees
- moved C21 1.55 mm to (132.2, 121.3), turned to 90 degrees
- moved C24 1.14 mm to (126.1, 113.2), turned to 180 degrees
- moved C19 1.02 mm to (133.7, 125.9)
- moved R25 1.02 mm to (133.7, 122.9)
- moved U4 1.02 mm to (130.7, 124.6)
- moved C16 1.02 mm to (136.8, 118.3)
- moved L3 1.02 mm to (130.7, 127.9)
- moved C17 0.76 mm to (136.8, 121.3)
- moved C22 0.72 mm to (126.1, 116.3), turned to 180 degrees
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Connections:
- J1 pad A12: GND -> (no net)
- J1 pad A5: Net-(J1-PadA5) -> (no net)
- J1 pad A9: VBUS -> (no net)
- J1 pad B12: GND -> (no net)
- J1 pad B5: Net-(J1-PadB5) -> (no net)
- J1 pad B9: VBUS -> (no net)
- J1 pad S1: GND -> (no net)
Routing:
- net +3.3V: track 0.00 -> 22.2 mm
- net +5V: track 0.00 -> 18.5 mm
- net Net-(R25-Pad1): track 0.00 -> 4.34 mm
- net Net-(R24-Pad1): track 0.00 -> 4.34 mm
- net Net-(R28-Pad1): track 0.00 -> 3.32 mm
- net Net-(R26-Pad1): track 0.00 -> 3.32 mm
- net Net-(C21-Pad1): track 0.00 -> 2.59 mm
- net Net-(C20-Pad1): track 0.00 -> 2.59 mm
- net GND: vias 6 -> 4
