File: Hardware/PCB/BatteryBoard/BatteryBoard-backups/BatteryBoard-2023-12-28_211333/BatteryBoard.kicad_sch (KiCad schematic)
At the start: 77 parts, among them J1 USB_C_Receptacle_USB2.0, J2 Thermistor, J3 Conn_01x07, J4 Conn_01x07, J5 Conn_01x07, J6 Conn_01x07, J7 Power, Q1 FDS4935A, Q2 FDS4935A, SW1 SW_SPDT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

Commit message: 配線中
Parts:
- C22, C23: value 10u(3216) -> 10u(3225); footprint Capacitor_SMD:C_1206_3216Metric -> Capacitor_SMD:C_1210_3225Metric
- C24, C25: value 22u(3216) -> 22u(3225); footprint Capacitor_SMD:C_1206_3216Metric -> Capacitor_SMD:C_1210_3225Metric
Changed lines of the file:
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@@
     (in_bom yes) (on_board yes)
     (property "Reference" "C23" (id 0) (at 255.27 113.03 0))
-    (property "Value" "10u(3216)" (id 1) (at 252.73 104.14 0))
-    (property "Footprint" "Capacitor_SMD:C_1206_3216Metric" (id 2) (at 252.73 111.76 0)
+    (property "Value" "10u(3225)" (id 1) (at 252.73 104.14 0))
+    (property "Footprint" "Capacitor_SMD:C_1210_3225Metric" (id 2) (at 252.73 111.76 0)
       (effects (font (size 1.27 1.27)) hide)
     )
@@
     (in_bom yes) (on_board yes)
     (property "Reference" "C25" (id 0) (at 260.35 113.03 0))
-    (property "Value" "22u(3216)" (id 1) (at 257.81 106.68 0))
-    (property "Footprint" "Capacitor_SMD:C_1206_3216Metric" (id 2) (at 257.81 111.76 0)
+    (property "Value" "22u(3225)" (id 1) (at 257.81 106.68 0))
+    (property "Footprint" "Capacitor_SMD:C_1210_3225Metric" (id 2) (at 257.81 111.76 0)
       (effects (font (size 1.27 1.27)) hide)
     )
@@
     (in_bom yes) (on_board yes)
     (property "Reference" "C24" (id 0) (at 260.35 73.66 0))
-    (property "Value" "22u(3216)" (id 1) (at 257.81 67.31 0))
-    (property "Footprint" "Capacitor_SMD:C_1206_3216Metric" (id 2) (at 257.81 72.39 0)
+    (property "Value" "22u(3225)" (id 1) (at 257.81 67.31 0))
+    (property "Footprint" "Capacitor_SMD:C_1210_3225Metric" (id 2) (at 257.81 72.39 0)
       (effects (font (size 1.27 1.27)) hide)
     )
@@
     (in_bom yes) (on_board yes)
     (property "Reference" "C22" (id 0) (at 255.27 73.66 0))
-    (property "Value" "10u(3216)" (id 1) (at 252.73 64.77 0))
-    (property "Footprint" "Capacitor_SMD:C_1206_3216Metric" (id 2) (at 252.73 72.39 0)
+    (property "Value" "10u(3225)" (id 1) (at 252.73 64.77 0))
+    (property "Footprint" "Capacitor_SMD:C_1210_3225Metric" (id 2) (at 252.73 72.39 0)
       (effects (font (size 1.27 1.27)) hide)
     )
@@
     )
     (path "/d98a0bdf-cc96-43af-9ff7-11bcaf3e8629"
-      (reference "C22") (unit 1) (value "10u(3216)") (footprint "Capacitor_SMD:C_1206_3216Metric")
+      (reference "C22") (unit 1) (value "10u(3225)") (footprint "Capacitor_SMD:C_1210_3225Metric")
     )
     (path "/4868940f-adc2-4f2b-af1e-d07b4458b722"
-      (reference "C23") (unit 1) (value "10u(3216)") (footprint "Capacitor_SMD:C_1206_3216Metric")
+      (reference "C23") (unit 1) (value "10u(3225)") (footprint "Capacitor_SMD:C_1210_3225Metric")
     )
     (path "/d6185a66-6f66-4600-b2df-1f313f971301"
-      (reference "C24") (unit 1) (value "22u(3216)") (footprint "Capacitor_SMD:C_1206_3216Metric")
+      (reference "C24") (unit 1) (value "22u(3225)") (footprint "Capacitor_SMD:C_1210_3225Metric")
     )
     (path "/8cec638d-b09e-414d-99c1-e1ec911f6775"
-      (reference "C25") (unit 1) (value "22u(3216)") (footprint "Capacitor_SMD:C_1206_3216Metric")
+      (reference "C25") (unit 1) (value "22u(3225)") (footprint "Capacitor_SMD:C_1210_3225Metric")
     )
     (path "/022a6323-f977-409c-beec-60bf89ec3424"
