File: Hardware/PCB/BatteryBoard/BatteryBoard-backups/BatteryBoard-2023-12-28_211333/BatteryBoard_old.kicad_sch (KiCad schematic)
At the start: 77 parts, among them J1 USB_C_Receptacle_USB2.0, J2 Thermistor, J3 Conn_01x07, J4 Conn_01x07, J5 Conn_01x07, J6 Conn_01x07, J7 Power, Q1 FDS4935A, Q2 FDS4935A, SW1 SW_SPDT, U1 BQ25887RGER, U2 LTC4417CGN, U3 TPS63070, U4 TPS63070

Commit message: 配線中
Parts:
- removed C1, C17: 10u(3225), Capacitor_SMD:C_1210_3225Metric, symbol Device:C_Small
- removed C11, C19, C2, C21, C3: 0.1u, Capacitor_SMD:C_0603_1608Metric, symbol Device:C_Small
- removed C23: 10u(3216), Capacitor_SMD:C_1206_3216Metric, symbol Device:C_Small
- removed C25: 22u(3216), Capacitor_SMD:C_1206_3216Metric, symbol Device:C_Small
- removed C30, C31: 4.7u, Capacitor_SMD:C_0805_2012Metric, symbol Device:C_Small
- removed L3: 1uH, Inductor_SMD:L_1210_3225Metric, symbol Device:L_Small
- removed Q2: FDS4935A, Package_SO:SOIC-8_3.9x4.9mm_P1.27mm, symbol Device:Q_Dual_PMOS_S1G1S2G2D2D2D1D1
- removed R1, R11, R12, R2, R3, R4, R5, R6, R7, R8: R_Small, Resistor_SMD:R_0603_1608Metric, symbol Device:R_Small
- removed R20: 240k, Resistor_SMD:R_0603_1608Metric, symbol Device:R_Small
- removed R25: 10k, Resistor_SMD:R_0603_1608Metric, symbol Device:R_Small
- removed R28: 470k, Resistor_SMD:R_0603_1608Metric, symbol Device:R_Small
- removed R29: 150k, Resistor_SMD:R_0603_1608Metric, symbol Device:R_Small
- removed U2: LTC4417CGN, Package_SO:SSOP-24_3.9x8.7mm_P0.635mm, symbol Power_Management:LTC4417CGN
- removed U4: TPS63070, Module_SparkFun_Buck-Boost:VQFN-15-HR(3X2.5), symbol Module_SparkFun_Buck-Boost:TPS63070
- added C7, C9: 1u, Capacitor_SMD:C_0603_1608Metric, symbol Device:C_Small
- added C? (x2): 10u(3225), Capacitor_SMD:C_1210_3225Metric, symbol Device:C_Small
- added C? (x2): 22u(3225), Capacitor_SMD:C_1210_3225Metric, symbol Device:C_Small
- added D3, D4: D_Schottky, CUHS20S30:CUHS20S30, symbol Device:D_Schottky
- added D?: D_Schottky_Small, symbol Device:D_Schottky_Small
- added Q2: BCV62, Package_TO_SOT_SMD:SOT-143, symbol Device:Q_Dual_PNP_C2C1E1E2
- added R13, R14, R16: 10k, Resistor_SMD:R_0603_1608Metric, symbol Device:R_Small
- added R15: 100, Resistor_SMD:R_0603_1608Metric, symbol Device:R_Small
- added R17, R18: k, Resistor_SMD:R_0603_1608Metric, symbol Device:R_Small
- added U2: NJW4190M, Kicad_Akiyuki_Footprint:DMP-8_P1.27mm, symbol NJW4190M:NJW4190M
- C8: value 0.1u -> 1u
- C?: renamed from C24; value 22u(3216) -> 22u(3225); footprint Capacitor_SMD:C_1206_3216Metric -> Capacitor_SMD:C_1210_3225Metric
- C?: renamed from C22; value 10u(3216) -> 10u(3225); footprint Capacitor_SMD:C_1206_3216Metric -> Capacitor_SMD:C_1210_3225Metric
- J5: renamed from J2; footprint Connector_JST:JST_PH_B2B-PH-K_1x02_P2.00mm_Vertical -> Connector_JST:JST_XH_B2B-XH-A_1x02_P2.50mm_Vertical
- R?: renamed from R26; value 680k -> 365k
- R?: renamed from R27; value 130k -> 68.1k
- U?: renamed from U3; footprint Module_SparkFun_Buck-Boost:VQFN-15-HR(3X2.5) -> SparkFun_Buck-Boost:VQFN-15-HR(3X2.5)
- renumbered C4 to C1, C5 to C2, C6 to C3, C7 to C4, C9 to C5, C10 to C6, C16 to C?, C20 to C?, C18 to C?, J3 to J1, J1 to J2, J4 to J3, J5 to J4, L2 to L?, R9 to R1, R21 to R10, R22 to R11, R23 to R12, R10 to R2, R13 to R3, R14 to R4, R15 to R5, R16 to R6, R17 to R7, R18 to R8, R19 to R9, R24 to R?
Connections:
- net +3.3V: now also R8.2, R9.2
- net +5V: now also R3.2, C?.1, C?.1, D?.1 (K)
- net +5VREF: no longer R3.2, R8.2, R9.2
- net +BATT: now also Q1.3 (S), D3.2 (A)
- net GND: now also C9.2, C?.2, C?.2, C?.2, C?.2, R13.2, R14.1, R16.1, R18.2, U2.5 (GND); no longer SW1.1 (A)
- net INT: now also J1.6 (Pin_6); no longer J1.7 (Pin_7)
- net PSEL: now also J1.7 (Pin_7); no longer J1.6 (Pin_6)
- net VBUS: now also C8.1, D?.2 (A), U2.3 (V+), U2.7 (ON/OFF); no longer Q1.5 (D), Q1.6 (G)
- net at SW1.2 (B): now also D4.1 (K), R15.2
- net at SW1.3 (C): now also D3.1 (K)
- net G1: no longer names the net of Q1.4 (G)
- net G1: now also R15.1; no longer Q1.2 (G)
- net VDD renamed VBAT
- net VBAT: now also Q1.1 (S), C?.1, C?.1, Q2.3 (E1); no longer Q1.7 (D), Q1.8 (G)
- removed net VS1: C8.1, Q1.1 (S), Q1.3 (S)
- new net: C7.1, U2.2 (C+)
- new net: C7.2, U2.4 (C-)
- new net: Q1.5 (D), Q1.6 (G), Q1.7 (D), Q1.8 (G), Q2.4 (E2)
- new net: Q2.1 (C2), R14.2
- new net: Q1.2 (G), Q2.2 (C1), R16.2
- new net: R13.1, SW1.1 (A)
- new net FB: R17.2, R18.1, U2.1 (FB)
- new net GATE: C9.1, D4.2 (A), R17.1, U2.8 (VOUT)
- no-connect marks 24 -> 20
Other:
- note added: "+5VREFはSTATとPGのプルアップとサーミスタに使えるが、敢えて使わない Max:50mA"
- note added: "Gate Driver"
- note added: "Ideal Diode"
- note added: "LEDが5Vか3V3かは 配線して決める"
- note added: "Switch"
- note added: "min:0V max:8.4V"
- note added: "フィードバック用抵抗は プルダウン抵抗を兼ねる"
- note removed: "+5VREF Max:50mA"
- note removed: "5V to 8.4V"
- note removed: "PowerPath Control"
- note removed: "USBが未接続でBQ25887がBATTから給電されている時に サーミスタ電源がVBUSでは使えないため、サーミスタ電源は5Vである必要がある。 LTC4417のENにスイッチを付けてオフにすると、 VBUSからBQ25887に給電、充電されるけど5Vサーミスタが使えないことになるので、 スイッチはBATT側につけてUVフォルトを作成する。"
- note removed: "Under/Over voltage fault"
- note removed: "出力コンデンサは BBコンバータの入力コンデンサと共有"
- moved on the sheet: C?, L?, Q1A, Q1B, R?, SW1, U?
