File: Hardware/PCB/BatteryBoard/BatteryBoard.kicad_pcb (KiCad board)
At the start: 4 copper layers, 60 x 60 mm, 80 parts, among them J1 USB_C_Receptacle_USB2.0, J2 Thermistor, J3 Conn_01x07, J4 Conn_01x07, J5 Conn_01x07, J6 Conn_01x07, J7 Power, Q1 FDS4935A, Q2 FDS4935A, SW1 SW_SPDT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

Commit message: 保護回路付きの18500が入るように変更
Parts:
- BT1, BT2: footprint Battery_extlib:BatteryClip_Keystone_18500 -> Battery_extlib:BatteryClip_Keystone_18500_Protected
- F1: value ASMDC300F/24-2 -> Polyfuse_Small
- moved F1 1.78 mm to (141.1, 107.1)
- moved G*** 0.63 mm to (146.2, 83.5)
Routing:
- net Net-(BT1-Pad2): track 27.4 -> 25.2 mm
- net VBAT: track 25.9 -> 28.0 mm
- net +BATT: track 30.0 -> 31.8 mm
- net GND: vias 241 -> 213

Commit message: 発注完了
Routing:
- net VDD: track 12.4 -> 13.7 mm
- net GND: vias 213 -> 215
Other:
- board text added: "1"
- board text added: "2"
- board text added: "20"
- board text added: "3"
- board text added: "4"
- board text added: "5"
- board text added: "6"
- board text added: "7"
- board text added: "8"

Commit message: 抵抗の値をKiCadPCBに反映
Parts:
- R1, R6: value R_Small -> 330k 0.1%
- R11: value R_Small -> 510k 5%
- R12: value R_Small -> 0
- R13: value 5.11k -> 5.1k 0.1%
- R14: value 30k -> 30k 0.1%
- R2: value R_Small -> 27k 0.1%
- R20: value 240k -> 390k 5%
- R21: value 374 -> 560 0.1%
- R26: value 680k -> 680k 5%
- R27: value 130k -> 130k 0.1%
- R28: value 470k -> 470k 5%
- R29: value 150k -> 150k 0.1%
- R3: value R_Small -> 75k 0.1%
- R4: value R_Small -> 68k 0.1%
- R5, R8: value R_Small -> 47k 0.1%
- R7: value R_Small -> 30k 0.1%
Changed lines of the file:
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@@
       (effects (font (size 1 1) (thickness 0.15)))
     )
-    (fp_text value "470k" (at 0 1.43 -270) (layer "F.Fab")
+    (fp_text value "470k 5%" (at 0 1.43 -270) (layer "F.Fab")
       (effects (font (size 1 1) (thickness 0.15)))
     )
@@
       (effects (font (size 1 1) (thickness 0.15)))
     )
-    (fp_text value "R_Small" (at 0 1.43 90) (layer "F.Fab")
+    (fp_text value "510k 5%" (at 0 1.43 90) (layer "F.Fab")
       (effects (font (size 1 1) (thickness 0.15)))
     )
@@
       (effects (font (size 1 1) (thickness 0.15)))
     )
-    (fp_text value "150k" (at 0 1.43 -270) (layer "F.Fab")
+    (fp_text value "150k 0.1%" (at 0 1.43 -270) (layer "F.Fab")
       (effects (font (size 1 1) (thickness 0.15)))
     )
@@
       (effects (font (size 0.8 1) (thickness 0.15)))
     )
-    (fp_text value "R_Small" (at 0 1.43 90) (layer "F.Fab")
+    (fp_text value "75k 0.1%" (at 0 1.43 90) (layer "F.Fab")
       (effects (font (size 1 1) (thickness 0.15)))
     )
@@
       (effects (font (size 0.8 1) (thickness 0.15)))
     )
-    (fp_text value "R_Small" (at 0 1.43 90) (layer "F.Fab")
+    (fp_text value "47k 0.1%" (at 0 1.43 90) (layer "F.Fab")
       (effects (font (size 1 1) (thickness 0.15)))
     )
@@
       (effects (font (size 1 1) (thickness 0.15)))
     )
-    (fp_text value "R_Small" (at 0 1.43 90) (layer "F.Fab")
+    (fp_text value "27k 0.1%" (at 0 1.43 90) (layer "F.Fab")
       (effects (font (size 1 1) (thickness 0.15)))
     )
@@
       (effects (font (size 1 1) (thickness 0.15)))
     )
-    (fp_text value "240k" (at 0 1.43 90) (layer "F.Fab")
+    (fp_text value "390k 5%" (at 0 1.43 90) (layer "F.Fab")
       (effects (font (size 1 1) (thickness 0.15)))
     )
@@
       (effects (font (size 1 0.8) (thickness 0.15)))
     )
-    (fp_text value "374" (at 0 1.43 -270) (layer "F.Fab")
+    (fp_text value "560 0.1%" (at 0 1.43 -270) (layer "F.Fab")
       (effects (font (size 1 1) (thickness 0.15)))
     )
@@
       (effects (font (size 0.8 1) (thickness 0.15)))
     )
-    (fp_text value "R_Small" (at 0 1.43 90) (layer "F.Fab")
+    (fp_text value "47k 0.1%" (at 0 1.43 90) (layer "F.Fab")
       (effects (font (size 1 1) (thickness 0.15)))
     )
@@
       (effects (font (size 1 1) (thickness 0.15)))
     )
-    (fp_text value "R_Small" (at 0 1.43 90) (layer "F.Fab")
+    (fp_text value "330k 0.1%" (at 0 1.43 90) (layer "F.Fab")
       (effects (font (size 1 1) (thickness 0.15)))
     )
@@
       (effects (font (size 1 1) (thickness 0.15)))
     )
-    (fp_text value "R_Small" (at 0 1.43 90) (layer "F.Fab")
+    (fp_text value "330k 0.1%" (at 0 1.43 90) (layer "F.Fab")
       (effects (font (size 1 1) (thickness 0.15)))
     )
@@
       (effects (font (size 1 0.8) (thickness 0.15)))
     )
-    (fp_text value "5.11k" (at 0 1.43 90) (layer "F.Fab")
+    (fp_text value "5.1k 0.1%" (at 0 1.43 90) (layer "F.Fab")
       (effects (font (size 1 1) (thickness 0.15)))
     )
@@
       (effects (font (size 1 1) (thickness 0.15)))
     )
-    (fp_text value "680k" (at 0 1.43 -270) (layer "F.Fab")
+    (fp_text value "680k 5%" (at 0 1.43 -270) (layer "F.Fab")
       (effects (font (size 1 1) (thickness 0.15)))
     )
@@
       (effects (font (size 1 1) (thickness 0.15)))
     )
-    (fp_text value "R_Small" (at 0 1.43 90) (layer "F.Fab")
+    (fp_text value "0" (at 0 1.43 90) (layer "F.Fab")
       (effects (font (size 1 1) (thickness 0.15)))
     )
@@
       (effects (font (size 0.8 1) (thickness 0.15)))
     )
-    (fp_text value "R_Small" (at 0 1.43 90) (layer "F.Fab")
+    (fp_text value "68k 0.1%" (at 0 1.43 90) (layer "F.Fab")
       (effects (font (size 1 1) (thickness 0.15)))
     )
@@
       (effects (font (size 1 1) (thickness 0.15)))
     )
-    (fp_text value "30k" (at 0 1.43 90) (layer "F.Fab")
+    (fp_text value "30k 0.1%" (at 0 1.43 90) (layer "F.Fab")
       (effects (font (size 1 1) (thickness 0.15)))
     )
@@
       (effects (font (size 0.8 1) (thickness 0.15)))
     )
-    (fp_text value "R_Small" (at 0 1.43 90) (layer "F.Fab")
+    (fp_text value "30k 0.1%" (at 0 1.43 90) (layer "F.Fab")
       (effects (font (size 1 1) (thickness 0.15)))
     )
@@
       (effects (font (size 1 1) (thickness 0.15)))
     )
-    (fp_text value "130k" (at 0 1.43 -270) (layer "F.Fab")
+    (fp_text value "130k 0.1%" (at 0 1.43 -270) (layer "F.Fab")
       (effects (font (size 1 1) (thickness 0.15)))
     )
