File: Hardware/PCB/CommunicationBoard/CommunicationBoard.kicad_sch (KiCad schematic)
At the start: 48 parts, among them J1 SWD, J2 Conn_01x07, J3 Conn_01x07, J4 Conn_01x07, J6 USB_C_Receptacle_USB2.0, J7 TWELITER, SW1 nRF_RESET, SW2 nRF_DFU, SW3 TWE_CLEAR, SW4 TWE_RESET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

Commit message: 回路図を微修正、基板を更新済み
Parts:
- removed U6: MW-R-DP-W, Package_DIP:DIP-28_W15.24mm, symbol RF_ZigBee:MW-R-DP-W
- added R16: DNF, Resistor_SMD:R_0603_1608Metric, symbol Device:R_Small
- JP1, JP2, JP3: renamed from JP?; footprint (none) -> Jumper:SolderJumper-2_P1.3mm_Open_RoundedPad1.0x1.5mm
- gave numbers to parts that had none: 2
Connections:
- net GND: now also R16.2
- net at U5.17 (DIO15/SDA), U7.4: now also R16.1
Other:
- note added: "M1をGNDへ接続すると親機、開放またはVCCへ接続すると子機 フラッシュクリア時、M1 は Hiまたはオープン ->インタラクティブモードで解決"
- note removed: "M1をGNDへ接続すると親機、開放またはVCCへ接続すると子機として使用できます。 フラッシュクリア時、M1 は Hiまたはオープン"

Commit message: 無線ボード配線7割
Parts:
- added C10, C9: 10μF35V X5R 2012, Capacitor_SMD:C_0805_2012Metric, symbol Device:C_Small
Connections:
- net +3.3V: now also C10.1, C9.1
- net GND: now also C10.2, C9.2
- net SEL0: now also U3.19 (P0_29_AIN5); no longer U3.12 (P0_04_AIN2)
- net SEL1: now also U3.20 (P0_28_AIN4); no longer U3.13 (P0_03_AIN1)
- removed net +5V: J2.1 (Pin_1), J3.1 (Pin_1), J4.1 (Pin_1)
- no-connect marks 33 -> 36
Other:
- moved on the sheet: J2, J3, J4

Commit message: 残り未配線23
Connections:
- net +3.3V: no longer J3.3 (Pin_3), J4.3 (Pin_3)
- net GND: no longer J3.2 (Pin_2), J4.2 (Pin_2)
- net TWE_UART_RTS: now also U3.13 (P0_03_AIN1); no longer U3.16 (P0_02_AIN0)
- no-connect marks 36 -> 40
Changed lines of the file:
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@@
   (junction (at 111.76 146.05) (diameter 0) (color 0 0 0 0)
   )
+  (no_connect (at 91.44 40.64))
   (no_connect (at 228.6 52.07))
   (no_connect (at 148.59 138.43))
@@
   (no_connect (at 68.58 27.94))
   (no_connect (at 147.32 85.09))
+  (no_connect (at 91.44 38.1))
   (no_connect (at 229.87 87.63))
   (no_connect (at 148.59 140.97))
   (no_connect (at 45.72 158.75))
+  (no_connect (at 68.58 40.64))
   (no_connect (at 148.59 118.11))
   (no_connect (at 45.72 166.37))
@@
   (no_connect (at 184.15 125.73))
   (no_connect (at 91.44 43.18))
+  (no_connect (at 68.58 38.1))
   (no_connect (at 228.6 54.61))
-  (no_connect (at 45.72 168.91))
   (no_connect (at 184.15 120.65))
   (no_connect (at 45.72 143.51))
   (no_connect (at 91.44 35.56))
+  (no_connect (at 71.12 186.69))
   (no_connect (at 68.58 35.56))
   (no_connect (at 91.44 27.94))
@@
     (stroke (width 0) (type default) (color 0 0 0 0))
   )
+  (wire (pts (xy 40.64 168.91) (xy 45.72 168.91))
+    (stroke (width 0) (type default) (color 0 0 0 0))
+  )
   (wire (pts (xy 135.89 30.48) (xy 137.16 30.48))
     (stroke (width 0) (type default) (color 0 0 0 0))
@@
     (effects (font (size 1.27 1.27)) (justify right bottom))
   )
+  (label "TWE_UART_RTS" (at 40.64 168.91 180)
+    (effects (font (size 1.27 1.27)) (justify right bottom))
+  )
   (label "TWE_UART_RTS" (at 184.15 128.27 0)
     (effects (font (size 1.27 1.27)) (justify left bottom))
@@
   (label "CH340K_TXD" (at 245.11 82.55 0)
     (effects (font (size 1.27 1.27)) (justify left bottom))
-  )
-  (label "TWE_UART_RTS" (at 71.12 186.69 270)
-    (effects (font (size 1.27 1.27)) (justify right bottom))
   )
   (label "FRST" (at 45.72 151.13 180)
@@
       (effects (font (size 1.016 1.016)) (justify left) hide)
     )
-  )
-  (symbol (lib_id "power:+3.3V") (at 91.44 38.1 270) (unit 1)
-    (in_bom yes) (on_board yes)
-    (property "Reference" "#PWR026" (id 0) (at 87.63 38.1 0)
-      (effects (font (size 1.27 1.27)) hide)
-    )
-    (property "Value" "+3.3V" (id 1) (at 93.98 38.1 90)
-      (effects (font (size 1.27 1.27)) (justify left))
-    )
-    (property "Footprint" "" (id 2) (at 91.44 38.1 0)
-      (effects (font (size 1.27 1.27)) hide)
-    )
-    (property "Datasheet" "" (id 3) (at 91.44 38.1 0)
-      (effects (font (size 1.27 1.27)) hide)
-    )
-    (pin "1")
   )
   (symbol (lib_id "power:+3.3V") (at 232.41 73.66 0) (unit 1)
@@
     )
     (property "Datasheet" "" (id 3) (at 209.55 151.13 0)
-      (effects (font (size 1.27 1.27)) hide)
-    )
-    (pin "1")
-  )
-  (symbol (lib_id "power:GND") (at 68.58 40.64 90) (unit 1)
-    (in_bom yes) (on_board yes)
-    (property "Reference" "#PWR024" (id 0) (at 74.93 40.64 0)
-      (effects (font (size 1.27 1.27)) hide)
-    )
-    (property "Value" "GND" (id 1) (at 71.12 40.64 90)
-      (effects (font (size 1.27 1.27)) (justify right))
-    )
-    (property "Footprint" "" (id 2) (at 68.58 40.64 0)
-      (effects (font (size 1.27 1.27)) hide)
-    )
-    (property "Datasheet" "" (id 3) (at 68.58 40.64 0)
       (effects (font (size 1.27 1.27)) hide)
     )
@@
     (pin "1")
   )
-  (symbol (lib_id "power:GND") (at 91.44 40.64 90) (unit 1)
-    (in_bom yes) (on_board yes)
-    (property "Reference" "#PWR027" (id 0) (at 97.79 40.64 0)
-      (effects (font (size 1.27 1.27)) hide)
-    )
-    (property "Value" "GND" (id 1) (at 93.98 40.64 90)
-      (effects (font (size 1.27 1.27)) (justify right))
-    )
-    (property "Footprint" "" (id 2) (at 91.44 40.64 0)
-      (effects (font (size 1.27 1.27)) hide)
-    )
-    (property "Datasheet" "" (id 3) (at 91.44 40.64 0)
-      (effects (font (size 1.27 1.27)) hide)
-    )
-    (pin "1")
-  )
   (symbol (lib_id "Jumper:SolderJumper_2_Open") (at 128.27 148.59 0) (unit 1)
     (in_bom yes) (on_board yes)
@@
     (pin "1")
     (pin "2")
-  )
-  (symbol (lib_id "power:+3.3V") (at 68.58 38.1 270) (unit 1)
-    (in_bom yes) (on_board yes)
-    (property "Reference" "#PWR023" (id 0) (at 64.77 38.1 0)
-      (effects (font (size 1.27 1.27)) hide)
-    )
-    (property "Value" "+3.3V" (id 1) (at 71.12 38.1 90)
-      (effects (font (size 1.27 1.27)) (justify left))
-    )
-    (property "Footprint" "" (id 2) (at 68.58 38.1 0)
-      (effects (font (size 1.27 1.27)) hide)
-    )
-    (property "Datasheet" "" (id 3) (at 68.58 38.1 0)
-      (effects (font (size 1.27 1.27)) hide)
-    )
-    (pin "1")
   )
   (symbol (lib_id "Connector:Conn_ARM_JTAG_SWD_10") (at 134.62 80.01 0) (unit 1)
@@
       (reference "#PWR021") (unit 1) (value "GND") (footprint "")
     )
-    (path "/b96e8e7e-0489-4502-b153-2b4cbf0e2890"
-      (reference "#PWR023") (unit 1) (value "+3.3V") (footprint "")
-    )
-    (path "/46f3665f-7e4a-4450-bf9b-92a5a5e94a65"
-      (reference "#PWR024") (unit 1) (value "GND") (footprint "")
-    )
-    (path "/0070ec71-f48d-469c-b7e9-a8aab28fc92d"
-      (reference "#PWR026") (unit 1) (value "+3.3V") (footprint "")
-    )
-    (path "/b450d685-ae0c-4286-9ce1-1f24b344dd02"
-      (reference "#PWR027") (unit 1) (value "GND") (footprint "")
-    )
     (path "/1414168c-ff98-4545-ab0f-ddcf59856a67"

Commit message: 未配線0
Connections:
- net P0.15: no longer names the net of J2.7 (Pin_7)
- net P0.15: no longer U3.43 (P0_15/TRCDAT2)
- net P0.16: no longer names the net of J2.6 (Pin_6)
- net P0.16: no longer U3.42 (P0_16/TRCDAT1)
- no-connect marks 40 -> 44
Changed lines of the file:
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@@
   (no_connect (at 73.66 186.69))
   (no_connect (at 184.15 135.89))
+  (no_connect (at 71.12 123.19))
   (no_connect (at 45.72 163.83))
   (no_connect (at 30.48 43.18))
@@
   (no_connect (at 91.44 35.56))
   (no_connect (at 71.12 186.69))
+  (no_connect (at 30.48 30.48))
   (no_connect (at 68.58 35.56))
   (no_connect (at 91.44 27.94))
@@
   (no_connect (at 233.68 43.18))
   (no_connect (at 91.44 30.48))
+  (no_connect (at 73.66 123.19))
   (no_connect (at 68.58 33.02))
   (no_connect (at 209.55 87.63))
   (no_connect (at 45.72 153.67))
+  (no_connect (at 30.48 27.94))
   (no_connect (at 184.15 130.81))
   (no_connect (at 45.72 146.05))
@@
     (stroke (width 0) (type default) (color 0 0 0 0))
   )
-  (wire (pts (xy 73.66 118.11) (xy 67.31 118.11))
-    (stroke (width 0) (type default) (color 0 0 0 0))
-  )
   (wire (pts (xy 127 130.81) (xy 124.46 130.81))
     (stroke (width 0) (type default) (color 0 0 0 0))
@@
     (stroke (width 0) (type default) (color 0 0 0 0))
   )
-  (wire (pts (xy 73.66 123.19) (xy 73.66 118.11))
-    (stroke (width 0) (type default) (color 0 0 0 0))
-  )
   (wire (pts (xy 111.76 163.83) (xy 111.76 171.45))
     (stroke (width 0) (type default) (color 0 0 0 0))
@@
     (stroke (width 0) (type default) (color 0 0 0 0))
   )
-  (wire (pts (xy 71.12 120.65) (xy 67.31 120.65))
-    (stroke (width 0) (type default) (color 0 0 0 0))
-  )
   (wire (pts (xy 135.89 128.27) (xy 148.59 128.27))
     (stroke (width 0) (type default) (color 0 0 0 0))
@@
   )
   (wire (pts (xy 205.74 62.23) (xy 213.36 62.23))
-    (stroke (width 0) (type default) (color 0 0 0 0))
-  )
-  (wire (pts (xy 71.12 123.19) (xy 71.12 120.65))
     (stroke (width 0) (type default) (color 0 0 0 0))
   )
@@
     )
   )
-  (global_label "P0.15" (shape passive) (at 30.48 27.94 0) (fields_autoplaced)
-    (effects (font (size 1.016 1.016)) (justify left))
-    (property "Intersheet References" "${INTERSHEET_REFS}" (id 0) (at 36.8131 28.0035 0)
-      (effects (font (size 1.016 1.016)) (justify left) hide)
-    )
-  )
   (global_label "TWE_RX_SUB" (shape passive) (at 217.17 149.86 0) (fields_autoplaced)
     (effects (font (size 1.016 1.016)) (justify left))
@@
     )
   )
-  (global_label "P0.16" (shape passive) (at 30.48 30.48 0) (fields_autoplaced)
-    (effects (font (size 1.016 1.016)) (justify left))
-    (property "Intersheet References" "${INTERSHEET_REFS}" (id 0) (at 36.8131 30.5435 0)
-      (effects (font (size 1.016 1.016)) (justify left) hide)
-    )
-  )
   (global_label "TWE_RX_SUB" (shape passive) (at 93.98 78.74 0) (fields_autoplaced)
     (effects (font (size 1.016 1.016)) (justify left))
@@
     )
   )
-  (global_label "P0.15" (shape passive) (at 67.31 120.65 180) (fields_autoplaced)
-    (effects (font (size 1.016 1.016)) (justify right))
-    (property "Intersheet References" "${INTERSHEET_REFS}" (id 0) (at 60.9769 120.5865 0)
-      (effects (font (size 1.016 1.016)) (justify right) hide)
-    )
-  )
   (global_label "PICO_RX" (shape passive) (at 30.48 33.02 0) (fields_autoplaced)
     (effects (font (size 1.016 1.016)) (justify left))
@@
     )
   )
-  (global_label "P0.16" (shape passive) (at 67.31 118.11 180) (fields_autoplaced)
-    (effects (font (size 1.016 1.016)) (justify right))
-    (property "Intersheet References" "${INTERSHEET_REFS}" (id 0) (at 60.9769 118.0465 0)
-      (effects (font (size 1.016 1.016)) (justify right) hide)
-    )
-  )
