File: Hardware/PCB/MediaBoard/MediaBoard.kicad_pcb (KiCad board)
At the start: 4 copper layers, 60 x 60 mm, 49 parts, among them J1 Conn_01x07, J2 Conn_01x07, J3 Micro_SD_Card_Det_Hirose_DM3AT, J4 Conn_01x07, J5 Conn_01x07, J6 RGBLED, U1 RaspberryPi-Pico, U2 MAX98357

Commit message: もろもろ更新
Parts:
- U1: value RaspberryPi-Pico -> WisdPi_Tiny_RP2040; footprint Module_extlib:RaspberryPi-Pico -> Module_extlib:WisdPi_Tiny_RP2040
- moved J6 75.1 mm to (143.0, 133.1)
- moved LS1 69.9 mm to (167.9, 99.5), turned to 90 degrees
- moved C3 48.5 mm to (120.6, 107.1), turned to 90 degrees
- moved C5 43.9 mm to (123.7, 107.1), turned to 90 degrees
- moved R5 35.7 mm to (159.2, 89.3), turned to 180 degrees
- moved R2 34.0 mm to (166.3, 89.3), turned to 180 degrees
- moved R6 30.1 mm to (156.2, 89.3)
- moved C4 29.9 mm to (162.3, 89.3)
- moved C1 28.7 mm to (162.3, 90.9)
- moved C7 25.9 mm to (152.1, 110.2)
- moved C12 24.1 mm to (144.5, 104.6)
- moved C13 22.8 mm to (144.5, 106.1)
- moved U2 22.1 mm to (143.5, 101.5)
- moved C9 21.4 mm to (152.1, 117.3)
- moved D2 20.8 mm to (147.0, 110.7)
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Connections:
- U1 pad 10: unconnected-(U1-Pad10) -> Net-(R7-Pad1)
- U1 pad 11: unconnected-(U1-Pad11) -> Net-(R8-Pad1)
- U1 pad 12: Net-(R7-Pad1) -> Net-(R9-Pad1)
- U1 pad 13: GND -> unconnected-(U1-Pad13)
- U1 pad 14: Net-(R8-Pad1) -> unconnected-(U1-Pad14)
- U1 pad 15: Net-(R9-Pad1) -> unconnected-(U1-Pad15)
- U1 pad 17: unconnected-(U1-Pad17) -> /MISO0
- U1 pad 18: GND -> /CS0
- U1 pad 19: unconnected-(U1-Pad19) -> /SCK0
- U1 pad 20: unconnected-(U1-Pad20) -> /MOSI0
- U1 pad 21: /MISO0 -> unconnected-(U1-Pad21)
- U1 pad 22: /CS0 -> unconnected-(U1-Pad22)
- U1 pad 23: GND -> unconnected-(U1-Pad23)
- U1 pad 24: /SCK0 -> unconnected-(U1-Pad24)
- U1 pad 25: /MOSI0 -> unconnected-(U1-Pad25)
- U1 pad 27: unconnected-(U1-Pad27) -> +3.3V
- U1 pad 3: GND -> unconnected-(U1-Pad3)
- U1 pad 8: GND -> unconnected-(U1-Pad8)
